File: KiCad/Main Board/Electronic Target.sch (KiCad schematic (older format))
At the start: 51 parts, among them J1 Conn_02x06_Odd_Even, J2 Conn_02x04_Odd_Even, U1 LM75AIMX_NOPB, U2 74LV8154, U3 LM339, U4 74HC74, U5 74HC00, U6 74LV8154, U7 74HC74, U8 NMA0505SC, X1 8M0

Commit message: Revison 2.2 Data Aquisition
These are the schematics after board revisions.

Note, the Gerber files are no longer valid and have been removed.
Parts:
- added J6: Conn_01x06, symbol Connector_Generic:Conn_01x06
Connections:
- net labels added: ARX, ATX, PAPER, PAPER*, SPARE
- wire segments 354 -> 366
Changed lines of the file:
@@
 Title "freETarget"
 Date "2020-02-16"
-Rev "2.1.X"
+Rev "2.2"
 Comp "github.com/ten-point-nine/freETarget"
 Comment1 ""
@@
 $EndComp
 Connection ~ 3900 8400
+$Comp
+L Connector_Generic:Conn_01x06 J6
+U 1 1 5F996624
+P 800 3750
+F 0 "J6" H 718 4167 50  0000 C CNN
+F 1 "Conn_01x06" H 800 4100 50  0000 C CNN
+F 2 "" H 800 3750 50  0001 C CNN
+F 3 "~" H 800 3750 50  0001 C CNN
+	1    800  3750
+	-1   0    0    -1
+$EndComp
+$Comp
+L power:GND #PWR?
+U 1 1 5F9DF6CB
+P 1050 4300
+F 0 "#PWR?" H 1050 4050 50  0001 C CNN
+F 1 "GND" H 1055 4127 50  0000 C CNN
+F 2 "" H 1050 4300 50  0001 C CNN
+F 3 "" H 1050 4300 50  0001 C CNN
+	1    1050 4300
+	1    0    0    -1
+$EndComp
+$Comp
+L power:VCC #PWR?
+U 1 1 5F9E07B6
+P 1100 3250
+F 0 "#PWR?" H 1100 3100 50  0001 C CNN
+F 1 "VCC" H 1115 3423 50  0000 C CNN
+F 2 "" H 1100 3250 50  0001 C CNN
+F 3 "" H 1100 3250 50  0001 C CNN
+	1    1100 3250
+	1    0    0    -1
+$EndComp
+Wire Wire Line
+	1100 3250 1100 3550
+Wire Wire Line
+	1100 3550 1000 3550
+Wire Wire Line
+	1050 4050 1000 4050
+Wire Wire Line
+	1050 4050 1050 4300
+Wire Wire Line
+	1300 3950 1000 3950
+Wire Wire Line
+	1300 3750 1000 3750
+Wire Wire Line
+	15550 3700 15350 3700
+Wire Wire Line
+	15550 3800 15350 3800
+Wire Wire Line
+	15550 4100 15350 4100
+Wire Wire Line
+	15550 4200 15350 4200
+Text Label 15350 3700 0    50   ~ 0
+SPARE
+Text Label 15350 3800 0    50   ~ 0
+PAPER*
+Text Label 15350 4100 0    50   ~ 0
+ARX
+Text Label 15350 4200 0    50   ~ 0
+ATX
+Text Label 1050 3950 0    50   ~ 0
+PAPER
+Wire Wire Line
+	1000 3850 1300 3850
+Text Label 1050 3850 0    50   ~ 0
+SPARE
+Wire Wire Line
+	1000 3650 1300 3650
+Text Label 1050 3650 0    50   ~ 0
+ATX
+Text Label 1050 3750 0    50   ~ 0
+ARX
 $EndSCHEMATC

Commit message: Schematic  Revised to 2.2B
The LM339 was referenced to ground.  In practice the sound signal could go negative as much as 1.3VDC.  The absolute maximum rating for this value was -0.3VDC.  In practice the short negative voltage would cause a leakage current on the die and result in spurious outputs on the logic (timer start) lines.

This change puts the -V input to -5VDC so that the input signal is kept above the minimum signal value.
Parts:
- U1: symbol Electronic-Target-rescue:LM75AIMX_NOPB-2020-05-12_18-19-55 -> Electronic-Target-rescue:LM75AIMX_NOPB-2020-05-12_18-19-55-Electronic-Target-rescue
- U8: symbol Electronic-Target-rescue:NMA0505SC-NMA0505SC -> Electronic-Target-rescue:NMA0505SC-NMA0505SC-Electronic-Target-rescue
- XA1: symbol Electronic-Target-rescue:Arduino_Mega2560_Shield-arduino -> Electronic-Target-rescue:Arduino_Mega2560_Shield-arduino-Electronic-Target-rescue
Connections:
- wire segments 366 -> 365
Other:
- note added: "IMPORTANT\nV- is referenced to -5VDC"
- moved on the sheet: U3E, V-5
Changed lines of the file:
@@
 Sheet 1 1
 Title "freETarget"
-Date "2020-02-16"
-Rev "2.2"
+Date "2021-01-25"
+Rev "2.2B"
 Comp "github.com/ten-point-nine/freETarget"
 Comment1 ""
@@
 	11900 2550 11900 2500
 $Comp
-L Electronic-Target-rescue:Arduino_Mega2560_Shield-arduino XA1
+L Electronic-Target-rescue:Arduino_Mega2560_Shield-arduino-Electronic-Target-rescue XA1
 U 1 1 5E539FDE
 P 14050 5650
@@
 Wire Wire Line
 	4150 6050 4450 6050
-$Comp
-L Comparator:LM339 U3
-U 5 1 5E66D255
-P 9500 9100
-F 0 "U3" H 9458 9146 50  0000 L CNN
-F 1 "LM339" H 9458 9055 50  0000 L CNN
-F 2 "" H 9450 9200 50  0001 C CNN
-F 3 "https://www.st.com/resource/en/datasheet/lm139.pdf" H 9550 9300 50  0001 C CNN
-	5    9500 9100
-	1    0    0    -1
-$EndComp
 Wire Wire Line
 	10850 8800 10850 8700
-Wire Wire Line
-	9400 8800 9400 8700
-Wire Wire Line
-	9400 8700 10050 8700
-Wire Wire Line
-	9400 9400 9400 9700
-Wire Wire Line
-	9400 9700 10050 9700
 $Comp
 L power:VCC #PWR013
@@
 Connection ~ 10850 9700
 Wire Wire Line
-	9400 8700 8900 8700
-Wire Wire Line
 	8900 8700 8900 9050
-Connection ~ 9400 8700
 Connection ~ 8900 9050
-Connection ~ 9400 9700
 Wire Wire Line
 	8900 9350 8900 9700
 Connection ~ 8900 9350
-Wire Wire Line
-	8900 9700 9400 9700
-$Comp
-L Electronic-Target-rescue:NMA0505SC-NMA0505SC U8
+$Comp
+L Electronic-Target-rescue:NMA0505SC-NMA0505SC-Electronic-Target-rescue U8
 U 1 1 5ED14650
 P 5350 9200
@@
 Connection ~ 6050 9350
 Wire Wire Line
-	1500 1800 1500 8400
-Wire Wire Line
-	3900 8400 3900 9200
-Wire Wire Line
 	4650 9100 4350 9100
-Connection ~ 3900 9200
 Connection ~ 4650 9550
-Wire Wire Line
-	1500 8400 3900 8400
 Wire Wire Line
 	3900 9200 4650 9200
@@
 Connection ~ 700  1700
 $Comp
-L Electronic-Target-rescue:LM75AIMX_NOPB-2020-05-12_18-19-55 U1
+L Electronic-Target-rescue:LM75AIMX_NOPB-2020-05-12_18-19-55-Electronic-Target-rescue U1
 U 1 1 5ED0FC30
 P 13400 1900
@@
 L Connector_Generic:Conn_01x01 V-5
 U 1 1 5EFA3B8D
-P 3900 8200
-F 0 "V-5" V 3864 8112 50  0000 R CNN
-F 1 "TP" V 3773 8112 50  0000 R CNN
-F 2 "Connector_PinHeader_2.54mm:PinHeader_1x01_P2.54mm_Vertical" H 3900 8200 50  0001 C CNN
-F 3 "~" H 3900 8200 50  0001 C CNN
-	1    3900 8200
+P 3000 7900
+F 0 "V-5" V 2964 7812 50  0000 R CNN
+F 1 "TP" V 2873 7812 50  0000 R CNN
+F 2 "Connector_PinHeader_2.54mm:PinHeader_1x01_P2.54mm_Vertical" H 3000 7900 50  0001 C CNN
+F 3 "~" H 3000 7900 50  0001 C CNN
+	1    3000 7900
 	0    -1   -1   0
 $EndComp
-Connection ~ 3900 8400
 $Comp
 L Connector_Generic:Conn_01x06 J6
@@
 Text Label 1050 3750 0    50   ~ 0
 ARX
+Wire Wire Line
+	8900 9700 10050 9700
+$Comp
+L Comparator:LM339 U3
+U 5 1 5E66D255
+P 4200 8200
+F 0 "U3" V 4158 8246 50  0000 L CNN
+F 1 "LM339" V 3961 8155 50  0000 L CNN
+F 2 "" H 4150 8300 50  0001 C CNN
+F 3 "https://www.st.com/resource/en/datasheet/lm139.pdf" H 4250 8400 50  0001 C CNN
+	5    4200 8200
+	0    1    1    0
+$EndComp
+Wire Wire Line
+	8900 8700 10050 8700
+Wire Wire Line
+	1500 8100 1500 1800
+Wire Wire Line
+	1500 8100 3000 8100
+Connection ~ 3000 8100
+Wire Wire Line
+	3000 8100 3900 8100
+Connection ~ 3900 9200
+Connection ~ 3900 8100
+Wire Wire Line
+	3900 8100 3900 9200
+Wire Wire Line
+	6050 9050 6050 8100
+Wire Wire Line
+	6050 8100 4500 8100
+Connection ~ 6050 9050
+Text Notes 4500 8000 0    50   ~ 0
+IMPORTANT\nV- is referenced to -5VDC
 $EndSCHEMATC
